File: PCB/rocket_pack-basic.brd (EAGLE design)
At the start: 24.9 x 43.6 mm, 10 parts, among them U1 TPS73632_DBV_5, U2 LTC1540

Commit message: sleep timer and 'zero' header
Parts:
- moved R3 0.35 mm to (20.4, 51.3)
- turned AUX_POWER to 180 degrees
Routing:
- net VCC: track 28.6 -> 24.9 mm
- net GND: track 28.7 -> 28.6 mm, vias 2 -> 20
Other:
- board text added: "5.5V MAX"
- board text added: "Rocket Pack"
